Commit message: add sensor plugin

File: install/hanium_enu/share/hanium_enu/urdf/balancing_robot_urdf.urdf (robot description, URDF)
Before this commit: robot balancing_robot, 34 links, 33 joints
Joints:
- joint body_side_1__antenna_base_1: origin xyz=0.08710038582 0.000997190547 0.01825531893 rpy=2.653571843e-06 3.673205102e-06 1.570791437 -> xyz=-0.0009972294339 0.08710034819 0.0182556349 rpy=-3.673205093e-06 -1.349332362e-11 3.14158898
- joint body_side_1__body_bottom_1: origin xyz=-0.003786808445 -1.841649395e-08 0.002410168255 rpy=1.570793673 -3.673205102e-06 -1.570801217 -> xyz=3.184780997e-08 -0.003786744602 0.002409905552 rpy=1.5708 1.349343953e-11 -3.673205103e-06
- joint body_side_1__body_front_1_1: origin xyz=-0.0004107391661 0.0005002619865 0.06866082826 rpy=1.5708 -2.653571831e-06 3.141587764 -> xyz=-0.0005000092873 -0.0004110950825 0.06866058873 rpy=1.570796327 3.673205105e-06 -1.5708
- joint body_side_1__c_3_robot_export_clean_1__rx28_mount_1: origin xyz=-0.02527927186 0.0656147903 0.04780006482 rpy=1.570792654 2.653571827e-06 -4.889759748e-06 -> xyz=-0.06561458391 -0.025279575 0.04779990715 rpy=1.570796327 -3.673205108e-06 1.570792654
